File: hardware/octave-module/octave-module/octave-module.kicad_sch (KiCad schematic)
At the start: 26 parts, among them J1 JST_SH_4P, J2 JST_SH_4P

Commit message: Add octave-module flex PCB (fab-ready) + hardware to main
octave-module: uniform 13.708 mm LED pitch (caps aligned), solder lap-seam (J2 output / J3 input pads) with J2 plated 0.8 mm solder-access holes, full routing + GND pour, J1 placement; seam-lap footprint library; spacing/seam design docs; regenerated BOM + production files (J1 DNP, caps C14663, LEDs C2761795). Also controller_v2 + hardware BOM/docs.

Co-Authored-By: Claude Opus 4.8 <noreply@anthropic.com>
Parts:
- removed J2: JST_SH_4P, Connector_JST:JST_SH_SM04B-SRSS-TB_1x04-1MP_P1.00mm_Horizontal, symbol Connector:Conn_01x04_Socket
- added J2: Conn_01x03, seam-lap:Seam_LapPad_OUT_1x03, symbol Connector_Generic:Conn_01x03
- added J3: Conn_01x03, seam-lap:Seam_LapPad_IN_1x03, symbol Connector_Generic:Conn_01x03
- J1: value JST_SH_4P -> Conn_01x04_Socket
Connections:
- net DIN_PASS is gone; now on net GND: J1.4 (Pin_4)
- net +5V: now also J2.1 (Pin_1), J3.1 (Pin_1)
- net DIN_IN: now also J3.3 (Pin_3)
- net DOUT_OUT: now also J2.3 (Pin_3)
- net GND: now also J2.2 (Pin_2), J3.2 (Pin_2)
